File: hardware/kicad_design/design_1/design_1.kicad_pcb (KiCad board)
At the start: 4 copper layers, 85.4 x 157.2 mm, 145 parts, among them IC1 MIC7221YM5-TR, J1 Conn_01x02_Pin, J10 Conn_Coaxial, J11 Conn_Coaxial, J12 Conn_Coaxial, J13 Conn_Coaxial, J14 Barrel_Jack, J15 USB_C_Receptacle, J16 Conn_01x16_Pin, J3 Conn_02x07_Odd_Even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

Commit message: rev 5 board with termination resistors, through hole usb c, and minor fixes
Parts:
- removed J15: USB_C_Receptacle, handheld_mri_footprints:AMPHENOL_12401899E412A
- added J2: UJ31-CH-G2-SMT-TR, handheld_mri_footprints:CUI_UJ31-CH-G2-SMT-TR, F.Cu at (140.3, 166.8)
- added R17: 50, Resistor_SMD:R_0402_1005Metric, F.Cu at (94.1, 94.4)
- added R18: 50, Resistor_SMD:R_0402_1005Metric, F.Cu at (92.2, 94.4)
- added R19: 50, Resistor_SMD:R_0402_1005Metric, F.Cu at (96.0, 94.4)
- added R20: 50, Resistor_SMD:R_0402_1005Metric, F.Cu at (97.9, 94.4)
- added R21: 50, Resistor_SMD:R_0402_1005Metric, F.Cu at (99.8, 94.4)
- added R22: 50, Resistor_SMD:R_0402_1005Metric, F.Cu at (101.7, 94.4)
- added R23: 50, Resistor_SMD:R_0402_1005Metric, F.Cu at (103.6, 94.3)
- added R24: 50, Resistor_SMD:R_0402_1005Metric, F.Cu at (105.5, 94.3)
- moved R10 0.56 mm to (118.6, 168.6)
- moved R7 0.56 mm to (118.6, 167.7)
- moved H3 0.35 mm to (77.6, 36.5)
Routing:
- net /ft601/VBUS: track 64.0 -> 85.9 mm, vias 5 -> 4
- net GND: track 289.1 -> 297.6 mm, vias 335 -> 326
- net /ft601/CC1: track 23.3 -> 16.9 mm
- net /ft601/CC2: track 21.5 -> 18.0 mm, vias 2 -> 0
- net /ft601/RX2-: track 10.6 -> 8.46 mm
- net /ft601/RX2+: track 10.6 -> 8.46 mm
- net /ft601/TX1-: track 12.5 -> 10.4 mm
- net /ft601/TX1+: track 12.5 -> 10.4 mm
- net /ft601/D-: track 56.0 -> 57.7 mm
- net /ft601/RX1+: track 14.4 -> 12.8 mm, vias 2 -> 1
- net /ft601/TX2-: track 12.5 -> 10.9 mm, vias 2 -> 1
- net /ft601/TX2+: track 12.5 -> 10.9 mm, vias 2 -> 1
- net /ft601/D+: track 53.7 -> 55.2 mm
- net /ft601/RX1-: track 14.4 -> 13.0 mm, vias 2 -> 1
- net Net-(J5-In): track 76.1 -> 76.8 mm
Other:
- board text added: "AFE5812: Amplifiers & ADCs"
- board text added: "Streamoscope AFE5812 to Alchitry Au to FT601 Joseph Feld & Joe Steinmeyer Rev 5, August 2024"
- board text removed: "AFE5812: Amplifiers and ADCs"
- board text removed: "Streamoscope AFE5812 to Alchitry Au to FT601 Joseph Feld & Joe Steinmeyer Rev 4, July 2024"
